Commit message: Limit every joint to +/-45 degrees
The placeholder limits were +/-pi on the joints and +/-0.2 rad on the
springs. They are now +/-45 deg (0.7854 rad) on all 14 moving joints,
springs included, until the real mechanical stops are known.

The toe and heel frames keep their assumed spots, at the front and rear
edge of each sole: the switch positions are not final yet.

Co-Authored-By: Claude Opus 5 <noreply@anthropic.com>

File: zeus_description/urdf/zeus.urdf (robot description, URDF)
Before this commit: robot zeus, 35 links, 34 joints
Joints:
- joint left_ankle_pitch: limit lower=-3.1416 upper=3.1416 effort=25 velocity=20 -> lower=-0.7854 upper=0.7854 effort=25 velocity=20
- joint left_hip_pitch: limit lower=-3.1416 upper=3.1416 effort=25 velocity=20 -> lower=-0.7854 upper=0.7854 effort=25 velocity=20
- joint left_hip_pitch_spring: limit lower=-0.2 upper=0.2 effort=25 velocity=20 -> lower=-0.7854 upper=0.7854 effort=25 velocity=20
- joint left_hip_roll: limit lower=-3.1416 upper=3.1416 effort=25 velocity=20 -> lower=-0.7854 upper=0.7854 effort=25 velocity=20
- joint left_knee_pitch: limit lower=-3.1416 upper=3.1416 effort=25 velocity=20 -> lower=-0.7854 upper=0.7854 effort=25 velocity=20
- joint left_knee_pitch_spring: limit lower=-0.2 upper=0.2 effort=25 velocity=20 -> lower=-0.7854 upper=0.7854 effort=25 velocity=20
- joint right_ankle_pitch: limit lower=-3.1416 upper=3.1416 effort=25 velocity=20 -> lower=-0.7854 upper=0.7854 effort=25 velocity=20
- joint right_hip_pitch: limit lower=-3.1416 upper=3.1416 effort=25 velocity=20 -> lower=-0.7854 upper=0.7854 effort=25 velocity=20
- joint right_hip_pitch_spring: limit lower=-0.2 upper=0.2 effort=25 velocity=20 -> lower=-0.7854 upper=0.7854 effort=25 velocity=20
- joint right_hip_roll: limit lower=-3.1416 upper=3.1416 effort=25 velocity=20 -> lower=-0.7854 upper=0.7854 effort=25 velocity=20
- joint right_knee_pitch: limit lower=-3.1416 upper=3.1416 effort=25 velocity=20 -> lower=-0.7854 upper=0.7854 effort=25 velocity=20
- joint right_knee_pitch_spring: limit lower=-0.2 upper=0.2 effort=25 velocity=20 -> lower=-0.7854 upper=0.7854 effort=25 velocity=20
- joint waist_pitch: limit lower=-3.1416 upper=3.1416 effort=25 velocity=20 -> lower=-0.7854 upper=0.7854 effort=25 velocity=20
- joint waist_roll: limit lower=-3.1416 upper=3.1416 effort=25 velocity=20 -> lower=-0.7854 upper=0.7854 effort=25 velocity=20

Commit message: One foot switch per foot, at the centre of the sole
Each foot had two mechanical switches, at the toe and the heel, and the board
reported which of them was loaded. There is one per foot now, so that question
can no longer be asked: a foot is either taking weight or it is not.

Where the single switch sits is the whole decision, because that point is what
the InEKF pins the robot to while the foot is planted. The centre of the sole
is the least biased choice - either edge is a position the robot genuinely
stands on for only part of the stride, and anchoring there would bias the
estimate towards the phase when that end happens to be down. So the new
contact frame is the midpoint of the old toe and heel: x averaged, y and z the
sole itself, unchanged.

  zeus_model.yaml   left_toe/left_heel/right_toe/right_heel -> left_contact,
                    right_contact. zeus.urdf regenerated from it; the new
                    frame lands on the old midpoint to nine decimal places.
  clean_urdf.py     --suggest now measures the sole's centre, not its ends.
  NexusState.msg    contact[4] -> contact[2]. The two derived "this foot is
                    down" bits at 16 and 32 are gone: with one switch per foot
                    they would be copies of the switch bits.
  nexus_proto.py    v8 -> v9. The state packet loses 8 bytes, 434 -> 426, and
                    the policy block 46 floats -> 44. left_foot_down and
                    right_foot_down stay as named properties rather than
                    letting callers index contact[] - they read "either left
                    switch closed" before, and callers asking "is this foot
                    down" should not have to change again if a second switch
                    ever comes back.

The model test lost its toe-ahead-of-heel check along with the second frame.
What replaces it is the property that made the centre worth choosing: the
point sits near the middle of the sole, within 5 cm fore/aft of the ankle. A
model that silently kept the old toe frame passes every other check in that
file and fails this one.

Firmware side is a matching commit in stm32_zeuss; the two must be flashed and
deployed together, which is what the protocol version bump is for.

Co-Authored-By: Claude Opus 5 <noreply@anthropic.com>

File: zeus_description/urdf/zeus.urdf (robot description, URDF)
Before this commit: robot zeus, 35 links, 34 joints
Links:
- removed link left_heel
- removed link left_toe
- removed link right_heel
- removed link right_toe
- added link left_contact
- added link right_contact
Joints:
- removed joint left_foot_to_left_heel
- removed joint left_foot_to_left_toe
- removed joint right_foot_to_right_heel
- removed joint right_foot_to_right_toe
- added joint left_foot_to_left_contact: type fixed, parent left_foot, child left_contact, origin xyz=-0.00124329324 0.049748132 -0.0350954386 rpy=-1.56887986 -4.36180037e-05 -3.11883704
- added joint right_foot_to_right_contact: type fixed, parent right_foot, child right_contact, origin xyz=-0.00124602954 0.0498822512 0.0349044086 rpy=-1.56887986 -4.36180038e-05 -3.11883704
