Commit message: New CAD export: eight actuators, no waist in the model at all
A fresh Fusion export replaces the whole model - new meshes, new part names,
new axis convention. The important structural change is that it has no waist:
both hips bolt straight to the torso, where the previous export still carried
two waist joints that nothing drove.

The export arrived as mukesh.urdf, duplicated at two paths. It is a RAW export,
not a drop-in zeus.urdf: Fusion joint names, continuous joints with no limits,
no imu_link, no contact frames, robot name "leg_leg_leg". So it goes in as
urdf/zeus_raw.urdf, the pipeline's input, and zeus.urdf is generated from it as
before. The duplicate copy is gone.

zeus_model.yaml is rewritten against it:

  body frame   The export's handedness is the OPPOSITE of the last one: left is
               -X here and was +X, so forward becomes +Y. The check that this is
               right is that all twelve movable joints then land within 0.003 of
               a clean robot axis - ten pitch about +Y, two roll about +X. A
               wrong frame scatters them.
  links        Mapped by position in the kinematic chain, because the export
               mirrors parts without renaming them: each leg's two spring bodies
               carry the OTHER leg's side in their name. Same quirk as before.
  joints       Twelve: four drives and two springs a leg.
  imu          The export models the IMU board, so its position is measured
               rather than guessed at a box face as the old one had to be.

clean_urdf.py now SNAPS each axis to its declared direction instead of only
fixing its sign. The export carries 0.13 deg of skew on one leg and 0.26 on the
other; the legs disagreeing is what shows it to be export noise rather than
design intent, and left in it gives the two legs subtly different arcs for the
same joint angle.

WHICH LEG IS WHICH rests on the export's own link names, and cannot be checked
any other way: the new foot is exactly symmetric fore-and-aft - 210 mm long with
the ankle at its centre to within 2 mm - so there is no toe to point forward
with. If the robot ever behaves as though its legs are swapped, body_frame.left
is the first line to suspect.

THE IMU FRAME is declared robot-aligned, deliberately, even though the export
models the board yawed 90 degrees. imu_link is the frame the whole stack is
built on - the InEKF integrates in it, vel_hdg splits it into forward and
lateral, the policy is fed gyro in it - so yawing it turns "forward" into "left"
for all of them. Setting it to the modelled 90 degrees makes three host
kinematics assertions fail at once, which is the stack saying the same thing. If
the physical chip really is rotated, that rotation belongs in imu_bno085.c,
applied as the readings arrive. Unverified: hold the robot upright and read
imu_accel, which should be about (0, 0, +9.81).

BOLTED_JOINT_NAMES is now empty. It existed to put waist_pitch and waist_roll
into /joint_states at zero so robot_state_publisher could place the parts above
a waist the URDF had but nothing drove. There is no waist in the URDF now, and
naming a joint there that the model does not have would have it rejected on
every message.

Needs the matching stm32_zeuss commit: the firmware's kinematics drop from eight
joint angles per leg to six.

Co-Authored-By: Claude Opus 5 <noreply@anthropic.com>

File: zeus_description/urdf/zeus.urdf (robot description, URDF)
Before this commit: robot zeus, 33 links, 32 joints
Links:
- removed link left_hip_holder
- removed link left_knee_holder
- removed link left_knee_link
- removed link left_shin
- removed link left_thigh
- removed link pelvis
- removed link right_hip_holder
- removed link right_knee_holder
- removed link right_knee_link
- removed link right_shin
- removed link right_thigh
- removed link waist_bracket
- removed link waist_pitch_motor
- removed link waist_roll_motor
- added link imu_mount, mass 0.00700316929217391; collision mesh filename=package://zeus_description/meshes/IMU-1.stl scale=0.001 0.001 0.001; visual mesh filename=package://zeus_description/meshes/IMU-1.stl scale=0.001 0.001 0.001
- added link left_hip_bracket, mass 0.21747775609605063; collision mesh filename=package://zeus_description/meshes/hip_pitch_bracket_left.stl scale=0.001 0.001 0.001; visual mesh filename=package://zeus_description/meshes/hip_pitch_bracket_left.stl scale=0.001 0.001 0.001
- added link left_hip_roll_bracket, mass 0.2593952912339209; collision mesh filename=package://zeus_description/meshes/hip_roll_brackett_left.stl scale=0.001 0.001 0.001; visual mesh filename=package://zeus_description/meshes/hip_roll_brackett_left.stl scale=0.001 0.001 0.001
- added link left_knee_bracket, mass 0.2617120637060355; collision mesh filename=package://zeus_description/meshes/knee_brackett_left.stl scale=0.001 0.001 0.001; visual mesh filename=package://zeus_description/meshes/knee_brackett_left.stl scale=0.001 0.001 0.001
- added link right_hip_bracket, mass 0.21747775977773756; collision mesh filename=package://zeus_description/meshes/hip_pitch_bracket_right.s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 scale=0.001 0.001 0.001; visual mesh filename=package://zeus_description/meshes/hip_pitch_bracket_right.s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 scale=0.001 0.001 0.001
- added link right_hip_roll_bracket, mass 0.2593953363423353; collision mesh filename=package://zeus_description/meshes/Hip_roll_bracket_right.stl scale=0.001 0.001 0.001; visual mesh filename=package://zeus_description/meshes/Hip_roll_bracket_right.stl scale=0.001 0.001 0.001
- added link right_knee_bracket, mass 0.26171359081742096; collision mesh filename=package://zeus_description/meshes/knee_brackett_right.stl scale=0.001 0.001 0.001; visual mesh filename=package://zeus_description/meshes/knee_brackett_right.stl scale=0.001 0.001 0.001
- link left_ankle_motor: mass 0.5927007240078846 -> 0.7485386311285372; geometry collision mesh filename=package://zeus_description/meshes/Ankel_left.stl scale=0.001 0.001 0.001; visual mesh filename=package://zeus_description/meshes/Ankel_left.stl scale=0.001 0.001 0.001
- link left_foot: mass 0.25203061051460435 -> 0.24973822037059298; geometry collision mesh filename=package://zeus_description/meshes/foot_left.stl scale=0.001 0.001 0.001; visual mesh filename=package://zeus_description/meshes/foot_left.stl scale=0.001 0.001 0.001
- link left_hip_pitch_motor: mass 0.9354827862325781 -> 1.0900294297509525; geometry collision mesh filename=package://zeus_description/meshes/Hip_pitch_left.stl scale=0.001 0.001 0.001; visual mesh filename=package://zeus_description/meshes/Hip_pitch_left.stl scale=0.001 0.001 0.001
- link left_hip_roll_motor: mass 0.6149985412960198 -> 0.6101129224169122; geometry collision mesh filename=package://zeus_description/meshes/hip_roll_acc_left.stl scale=0.001 0.001 0.001; visual mesh filename=package://zeus_description/meshes/hip_roll_acc_left.stl scale=0.001 0.001 0.001
- link left_hip_spring: mass 0.04017905939509672 -> 0.07298374635894113; geometry collision mesh filename=package://zeus_description/meshes/Hip_spring_right.stl scale=0.001 0.001 0.001; visual mesh filename=package://zeus_description/meshes/Hip_spring_right.stl scale=0.001 0.001 0.001
- link left_knee_motor: mass 0.8362696907056681 -> 1.0350398151341045; geometry collision mesh filename=package://zeus_description/meshes/knee_actuator_left.stl scale=0.001 0.001 0.001; visual mesh filename=package://zeus_description/meshes/knee_actuator_left.stl scale=0.001 0.001 0.001
- link left_knee_spring: mass 0.04017905939509669 -> 0.0739166444341313; geometry collision mesh filename=package://zeus_description/meshes/Knee_spring_right.stl scale=0.001 0.001 0.001; visual mesh filename=package://zeus_description/meshes/Knee_spring_right.stl scale=0.001 0.001 0.001
- link right_ankle_motor: mass 0.5927007240078848 -> 0.748538133443455; geometry collision mesh filename=package://zeus_description/meshes/Ankel_right.stl scale=0.001 0.001 0.001; visual mesh filename=package://zeus_description/meshes/Ankel_right.stl scale=0.001 0.001 0.001
- link right_foot: mass 0.2520306105146048 -> 0.24973889755463174; geometry collision mesh filename=package://zeus_description/meshes/Foot_right.stl scale=0.001 0.001 0.001; visual mesh filename=package://zeus_description/meshes/Foot_right.stl scale=0.001 0.001 0.001
- link right_hip_pitch_motor: mass 0.9354827862325855 -> 1.0900294146990857; geometry collision mesh filename=package://zeus_description/meshes/Hip_pitch_right.stl scale=0.001 0.001 0.001; visual mesh filename=package://zeus_description/meshes/Hip_pitch_right.stl scale=0.001 0.001 0.001
- link right_hip_roll_motor: mass 0.6149985412960198 -> 0.6101127795645023; geometry collision mesh filename=package://zeus_description/meshes/hip_roll_acc_right.stl scale=0.001 0.001 0.001; visual mesh filename=package://zeus_description/meshes/hip_roll_acc_right.stl scale=0.001 0.001 0.001
- link right_hip_spring: mass 0.04017905939509668 -> 0.07298374635894113; geometry collision mesh filename=package://zeus_description/meshes/Hip_Spring_left.stl scale=0.001 0.001 0.001; visual mesh filename=package://zeus_description/meshes/Hip_Spring_left.stl scale=0.001 0.001 0.001
- link right_knee_motor: mass 0.836264992877475 -> 1.0350398163763748; geometry collision mesh filename=package://zeus_description/meshes/knee_right.stl scale=0.001 0.001 0.001; visual mesh filename=package://zeus_description/meshes/knee_right.stl scale=0.001 0.001 0.001
- link right_knee_spring: mass 0.04017905939509669 -> 0.0739166444341313; geometry collision mesh filename=package://zeus_description/meshes/Knee_spring_left.stl scale=0.001 0.001 0.001; visual mesh filename=package://zeus_description/meshes/Knee_spring_left.stl scale=0.001 0.001 0.001
- link torso: mass 0.4174748406112292 -> 0.6724614837537145
Joints:
- removed joint base_link_to_pelvis
- removed joint left_hip_holder_to_left_thigh
- removed joint left_knee_holder_to_left_knee_link
- removed joint left_knee_link_to_left_shin
- removed joint left_shin_to_left_ankle_motor
- removed joint left_thigh_to_left_knee_motor
- removed joint pelvis_to_left_hip_roll_motor
- removed joint pelvis_to_right_hip_roll_motor
- removed joint pelvis_to_waist_pitch_motor
- removed joint right_hip_holder_to_right_thigh
- removed joint right_knee_holder_to_right_knee_link
- removed joint right_knee_link_to_right_shin
- removed joint right_shin_to_right_ankle_motor
- removed joint right_thigh_to_right_knee_motor
- removed joint waist_bracket_to_waist_roll_motor
- removed joint waist_pitch
- removed joint waist_roll
- added joint base_link_to_torso: type fixed, parent base_link, child torso, origin xyz=0.00361362116 -0.0168814148 -0.554005521 rpy=0 0 -1.57079633
- added joint left_hip_bracket_to_left_hip_roll_motor: type fixed, parent left_hip_bracket, child left_hip_roll_motor, origin xyz=-0.07286658000000017 -0.017805650000000003 -0.08888396 rpy=-3.141592653589793 1.2037062152420227e-35 -1.3552527156068808e-20
- added joint left_hip_roll_bracket_to_left_knee_motor: type fixed, parent left_hip_roll_bracket, child left_knee_motor, origin xyz=-7.367000000000346e-05 -0.038659050000000014 -0.1758100700000001 rpy=3.1415926535897745 -1.0011929436545832e-18 2.704926097982091e-19
- added joint left_knee_bracket_to_left_ankle_motor: type fixed, parent left_knee_bracket, child left_ankle_motor, origin xyz=-0.22248103 0.0003116700000000125 -0.06936809000000001 rpy=-5.55107277147842e-17 -1.5707963267948963 0
- added joint right_hip_bracket_to_right_hip_roll_motor: type fixed, parent right_hip_bracket, child right_hip_roll_motor, origin xyz=-0.07312906000000012 0.018203900000000002 -0.08869976999999998 rpy=-3.141592653589793 6.07576109200659e-39 -1.3552527156068808e-20
- added joint right_hip_roll_bracket_to_right_knee_motor: type fixed, parent right_hip_roll_bracket, child right_knee_motor, origin xyz=0.0004410700000000034 0.03865789000000001 0.17581153000000002 rpy=1.9721522630525295e-31 -3.4512664603419266e-31 5.551115123125802e-17
- added joint right_knee_bracket_to_right_ankle_motor: type fixed, parent right_knee_bracket, child right_ankle_motor, origin xyz=-0.22240434999999997 -1.2490009027033011e-17 0.06958225999999999 rpy=5.551115123125783e-17 -1.5707963267948966 0
- added joint torso_to_imu_mount: type fixed, parent torso, child imu_mount, origin xyz=-0.025821939089959448 -0.012322293212967468 0.6806080832520717 rpy=-6.888251614786907e-05 0.0005516016747925701 -0.0022425458152757066
- added joint torso_to_left_hip_pitch_motor: type fixed, parent torso, child left_hip_pitch_motor, origin xyz=-0.0866735451213116 0.026559840567045447 0.6892580895544036 rpy=3.141523771073645 0.0005516016747925701 -0.0022425458152757066
- added joint torso_to_right_hip_pitch_motor: type fixed, parent torso, child right_hip_pitch_motor, origin xyz=0.05309447999821324 0.026587670011303938 0.6892580900028281 rpy=3.141523771073645 0.0005516016747925701 -0.0022425458152757066
- joint left_ankle_pitch: axis 0 -0.001917 -0.999998 -> -0.999997333 0.00224250593 0.000551754731; origin xyz=-0.00089221000000002 0.03505565 0.03493286999999995 rpy=0.0 -6.776263578034401e-21 3.469446951953614e-18 -> xyz=-0.038446619999999994 0.0001725500000000002 0.04804246 rpy=-2.1599340154984659e-19 -2.2171418266626333e-19 -2.130031436354674e-19
- joint left_foot_to_left_contact: origin xyz=-0.00124329324 0.049748132 -0.0350954386 rpy=-1.56887986 -4.36180037e-05 -3.11883704 -> xyz=0.0328232312 -0.00010520166 0.0900125516 rpy=3.1410409 6.7645352e-05 -1.57303887
- joint left_hip_pitch: axis 0.0019170000000000005 0.999998 6.776250025507247e-21 -> -0.999997333 -0.00224250593 -0.000551754731; origin xyz=0.07997929000000002 0.0016956900000000275 -0.06500337000000002 rpy=-1.5707963267948966 -0.0 -1.5707963267948966 -> xyz=0.026879780000000013 0.030117960000000013 0.06735187000000004 rpy=-3.141592653589793 -0.0 -1.1407813263841318e-19
- joint left_hip_pitch_spring: axis 0.0019170000000000005 0.999998 6.776250025507247e-21 -> -0.000551754731 0.00224250593 -0.999997333; child left_hip_holder -> left_hip_bracket; origin xyz=1.9169999999988363e-05 0.00999998000000005 0.0 rpy=0.0 -0.0 0.0 -> xyz=0.016499949999999996 3.7000000000000364e-05 9.110000000021046e-06 rpy=-3.141592653589793 -1.5707963267948966 0
- joint left_hip_roll: axis -0.999741 -0.022754 4.4e-05 -> -0.00224254359 0.999997483 6.7645352e-05; child left_hip_pitch_motor -> left_hip_roll_bracket; origin xyz=-0.03987371999999695 -0.03601130000000332 0.06591298999999999 rpy=1.5707963267948966 -2.1684043449710084e-19 -1.5707963267948124 -> xyz=-0.06300986000000008 0.02640298 -0.020051319999999997 rpy=1.2493735972000932e-19 1.5707963267948966 0
- joint left_knee_pitch: axis 0 -0.999998 0.001917 -> -0.999997333 -0.00224250593 -0.000551754731; origin xyz=-0.0017334400000000017 0.07213018000000006 0.06783976000000003 rpy=3.141592653589709 -0.0 0.0 -> xyz=0.05470685000000112 -0.00025463000000113504 0.06052262000000003 rpy=-3.1415926535897745 -2.0866038768906402e-30 1.112927950723139e-16
- joint left_knee_pitch_spring: axis 0.0019169999999999999 0.9999979999999999 0.0 -> -0.000551754731 0.00224250593 -0.999997333; child left_knee_holder -> left_knee_bracket; origin xyz=0.0 -0.010000009999999974 1.9169999999135712e-05 rpy=3.141592653589793 -1.5707963267947795 0 -> xyz=0.014999840000000014 6.727000000000206e-05 1.6549999999959653e-05 rpy=-3.141592653589793 -1.5707963267948966 0
- joint right_ankle_pitch: axis -1.3427179832402326e-20 -0.001917 -0.999998 -> -0.999997333 -0.00224250593 -0.000551754731; origin xyz=-0.0008922099999999844 -0.03492147 0.035067009999999996 rpy=-3.141592653589793 6.776263578034406e-21 -3.469446951953614e-18 -> xyz=0.0385 0.0 0.048 rpy=-3.141592653589793 -4.690812175909376e-31 8.154403576970184e-32
- joint right_foot_to_right_contact: origin xyz=-0.00124602954 0.0498822512 0.0349044086 rpy=-1.56887986 -4.36180038e-05 -3.11883704 -> xyz=-0.032691938 4.98163595e-05 -0.0901720268 rpy=-0.00055175476 -6.7645352e-05 1.57303887
- joint right_hip_pitch: axis 0.001917 0.999998 0 -> -0.999997333 0.00224250593 0.000551754731; origin xyz=0.07997929000000002 0.0019448899999999726 0.06499639000000001 rpy=-1.5707963267948966 -0.0 -1.5707963267948966 -> xyz=-0.026670080000000002 0.03023804000000001 0.06738140999999999 rpy=5.580160412282723e-19 1.0842021724855044e-19 -1.2763065979448198e-19
- joint right_hip_pitch_spring: axis 0.001917 0.999998 0 -> -0.000551754731 -0.00224250593 0.999997333; child right_hip_holder -> right_hip_bracket; origin xyz=-1.917000000005942e-05 -0.00999997999999998 0.0 rpy=0.0 -0.0 0.0 -> xyz=-0.01649996 3.699999999999981e-05 9.110000000021046e-06 rpy=3.141592653589793 1.5707963267948966 0
- joint right_hip_roll: axis -0.999741 -0.022754 4.4e-05 -> -0.00224254359 -0.999997483 -6.7645352e-05; child right_hip_pitch_motor -> right_hip_roll_bracket; origin xyz=-0.040126130000003 0.03601129999999657 0.06575964 rpy=1.5707963267948966 -2.1684043449710084e-19 1.570796326794981 -> xyz=-0.06254649000000008 -0.026193479999999995 -0.0201 rpy=1.9721522630525295e-31 -1.5707963267948966 0
- joint right_knee_pitch: axis 0 -0.999998 0.001917 -> -0.999997333 0.00224250593 0.000551754731; origin xyz=-0.0017334400000000017 0.07086956000000008 -0.06811389000000002 rpy=3.469446951953614e-18 2.407412430484045e-35 -6.93889390390723e-18 -> xyz=-0.05464062 -9.409999999999974e-06 0.060582960000000026 rpy=-2.4805977683707598e-31 -6.401791135143172e-31 -1.9311058811127647e-31
- joint right_knee_pitch_spring: axis 0.001917 -0.999998 0 -> -0.000551754731 0.00224250593 -0.999997333; child right_knee_holder -> right_knee_bracket; origin xyz=0.0 0.00999997999999998 -1.917000000002389e-05 rpy=6.932117640329194e-18 -1.5707963267948966 0 -> xyz=-0.014999999999999998 0.0 0.0 rpy=1.4791141972893971e-31 1.5707963267948966 0
- joint torso_to_imu_link: origin xyz=0.068814036 -0.00686923244 -0.140457673 rpy=-3.13967519 0.022755615 -3.14154902 -> xyz=-0.0155814148 -0.00361362116 0.681405521 rpy=0 0 1.57079633
