Commit message: New CAD export: eight actuators, no waist in the model at all
A fresh Fusion export replaces the whole model - new meshes, new part names,
new axis convention. The important structural change is that it has no waist:
both hips bolt straight to the torso, where the previous export still carried
two waist joints that nothing drove.

The export arrived as mukesh.urdf, duplicated at two paths. It is a RAW export,
not a drop-in zeus.urdf: Fusion joint names, continuous joints with no limits,
no imu_link, no contact frames, robot name "leg_leg_leg". So it goes in as
urdf/zeus_raw.urdf, the pipeline's input, and zeus.urdf is generated from it as
before. The duplicate copy is gone.

zeus_model.yaml is rewritten against it:

  body frame   The export's handedness is the OPPOSITE of the last one: left is
               -X here and was +X, so forward becomes +Y. The check that this is
               right is that all twelve movable joints then land within 0.003 of
               a clean robot axis - ten pitch about +Y, two roll about +X. A
               wrong frame scatters them.
  links        Mapped by position in the kinematic chain, because the export
               mirrors parts without renaming them: each leg's two spring bodies
               carry the OTHER leg's side in their name. Same quirk as before.
  joints       Twelve: four drives and two springs a leg.
  imu          The export models the IMU board, so its position is measured
               rather than guessed at a box face as the old one had to be.

clean_urdf.py now SNAPS each axis to its declared direction instead of only
fixing its sign. The export carries 0.13 deg of skew on one leg and 0.26 on the
other; the legs disagreeing is what shows it to be export noise rather than
design intent, and left in it gives the two legs subtly different arcs for the
same joint angle.

WHICH LEG IS WHICH rests on the export's own link names, and cannot be checked
any other way: the new foot is exactly symmetric fore-and-aft - 210 mm long with
the ankle at its centre to within 2 mm - so there is no toe to point forward
with. If the robot ever behaves as though its legs are swapped, body_frame.left
is the first line to suspect.

THE IMU FRAME is declared robot-aligned, deliberately, even though the export
models the board yawed 90 degrees. imu_link is the frame the whole stack is
built on - the InEKF integrates in it, vel_hdg splits it into forward and
lateral, the policy is fed gyro in it - so yawing it turns "forward" into "left"
for all of them. Setting it to the modelled 90 degrees makes three host
kinematics assertions fail at once, which is the stack saying the same thing. If
the physical chip really is rotated, that rotation belongs in imu_bno085.c,
applied as the readings arrive. Unverified: hold the robot upright and read
imu_accel, which should be about (0, 0, +9.81).

BOLTED_JOINT_NAMES is now empty. It existed to put waist_pitch and waist_roll
into /joint_states at zero so robot_state_publisher could place the parts above
a waist the URDF had but nothing drove. There is no waist in the URDF now, and
naming a joint there that the model does not have would have it rejected on
every message.

Needs the matching stm32_zeuss commit: the firmware's kinematics drop from eight
joint angles per leg to six.

Co-Authored-By: Claude Opus 5 <noreply@anthropic.com>

File: zeus_description/urdf/zeus_raw.urdf (robot description, URDF)
Before this commit: robot complete_bitch_shit, 29 links, 28 joints
Links:
- removed link Actuator-Knee-Right
- removed link Actuator-Left
- removed link Actuator-Right
- removed link Foot-Right
- removed link Foot-left
- removed link Hip-Left
- removed link Hip-Right
- removed link Hip-Roll-Actuator-Left
- removed link Hip-Roll-control-right
- removed link Hip-Spring-Left
- removed link Knee-Actuator-Left-1
- removed link Random-T
- removed link Shin-Right
- removed link Shin-left
- removed link Spring-Hip-Right
- removed link Spring-Knee-left
- removed link Spring-Right
- removed link Waist-Pitch-Actuator
- removed link Waist-Roll-Actuator
- removed link complete_actuator_decoy
- removed link complete_actuator_decoy-v7Mirror
- removed link holder_hip_2nd
- removed link holder_hip_2nd-1
- removed link holder_hip_2nd-v6Mirror
- removed link holder_hip_2ndMirror
- removed link knee_joint_2
- removed link knee_joint_2-v8Mirror
- removed link waist
- added link Ankel_left, mass 0.7485386311285372; collision mesh filename=meshes/Ankel_left.stl scale=0.001 0.001 0.001; visual mesh filename=meshes/Ankel_left.stl scale=0.001 0.001 0.001
- added link Ankel_right, mass 0.748538133443455; collision mesh filename=meshes/Ankel_right.stl scale=0.001 0.001 0.001; visual mesh filename=meshes/Ankel_right.stl scale=0.001 0.001 0.001
- added link Foot_right, mass 0.24973889755463174; collision mesh filename=meshes/Foot_right.stl scale=0.001 0.001 0.001; visual mesh filename=meshes/Foot_right.stl scale=0.001 0.001 0.001
- added link Hip_Spring_left, mass 0.07298374635894113; collision mesh filename=meshes/Hip_Spring_left.stl scale=0.001 0.001 0.001; visual mesh filename=meshes/Hip_Spring_left.stl scale=0.001 0.001 0.001
- added link Hip_pitch_left, mass 1.0900294297509525; collision mesh filename=meshes/Hip_pitch_left.stl scale=0.001 0.001 0.001; visual mesh filename=meshes/Hip_pitch_left.stl scale=0.001 0.001 0.001
- added link Hip_pitch_right, mass 1.0900294146990857; collision mesh filename=meshes/Hip_pitch_right.stl scale=0.001 0.001 0.001; visual mesh filename=meshes/Hip_pitch_right.stl scale=0.001 0.001 0.001
- added link Hip_roll_bracket_right, mass 0.2593953363423353; collision mesh filename=meshes/Hip_roll_bracket_right.stl scale=0.001 0.001 0.001; visual mesh filename=meshes/Hip_roll_bracket_right.stl scale=0.001 0.001 0.001
- added link Hip_spring_right, mass 0.07298374635894113; collision mesh filename=meshes/Hip_spring_right.stl scale=0.001 0.001 0.001; visual mesh filename=meshes/Hip_spring_right.stl scale=0.001 0.001 0.001
- added link IMU-1, mass 0.00700316929217391; collision mesh filename=meshes/IMU-1.stl scale=0.001 0.001 0.001; visual mesh filename=meshes/IMU-1.stl scale=0.001 0.001 0.001
- added link Knee_spring_left, mass 0.0739166444341313; collision mesh filename=meshes/Knee_spring_left.stl scale=0.001 0.001 0.001; visual mesh filename=meshes/Knee_spring_left.stl scale=0.001 0.001 0.001
- added link Knee_spring_right, mass 0.0739166444341313; collision mesh filename=meshes/Knee_spring_right.stl scale=0.001 0.001 0.001; visual mesh filename=meshes/Knee_spring_right.stl scale=0.001 0.001 0.001
- added link foot_left, mass 0.24973822037059298; collision mesh filename=meshes/foot_left.stl scale=0.001 0.001 0.001; visual mesh filename=meshes/foot_left.stl scale=0.001 0.001 0.001
- added link hip_pitch_bracket_left, mass 0.21747775609605063; collision mesh filename=meshes/hip_pitch_bracket_left.stl scale=0.001 0.001 0.001; visual mesh filename=meshes/hip_pitch_bracket_left.stl scale=0.001 0.001 0.001
- added link hip_pitch_bracket_right, mass 0.21747775977773756; collision mesh filename=meshes/hip_pitch_bracket_right.stl scale=0.001 0.001 0.001; visual mesh filename=meshes/hip_pitch_bracket_right.stl scale=0.001 0.001 0.001
- added link hip_roll_acc_left, mass 0.6101129224169122; collision mesh filename=meshes/hip_roll_acc_left.stl scale=0.001 0.001 0.001; visual mesh filename=meshes/hip_roll_acc_left.stl scale=0.001 0.001 0.001
- added link hip_roll_acc_right, mass 0.6101127795645023; collision mesh filename=meshes/hip_roll_acc_right.stl scale=0.001 0.001 0.001; visual mesh filename=meshes/hip_roll_acc_right.stl scale=0.001 0.001 0.001
- added link hip_roll_brackett_left, mass 0.2593952912339209; collision mesh filename=meshes/hip_roll_brackett_left.stl scale=0.001 0.001 0.001; visual mesh filename=meshes/hip_roll_brackett_left.stl scale=0.001 0.001 0.001
- added link knee_actuator_left, mass 1.0350398151341045; collision mesh filename=meshes/knee_actuator_left.stl scale=0.001 0.001 0.001; visual mesh filename=meshes/knee_actuator_left.stl scale=0.001 0.001 0.001
- added link knee_brackett_left, mass 0.2617120637060355; collision mesh filename=meshes/knee_brackett_left.stl scale=0.001 0.001 0.001; visual mesh filename=meshes/knee_brackett_left.stl scale=0.001 0.001 0.001
- added link knee_brackett_right, mass 0.26171359081742096; collision mesh filename=meshes/knee_brackett_right.stl scale=0.001 0.001 0.001; visual mesh filename=meshes/knee_brackett_right.stl scale=0.001 0.001 0.001
- added link knee_right, mass 1.0350398163763748; collision mesh filename=meshes/knee_right.stl scale=0.001 0.001 0.001; visual mesh filename=meshes/knee_right.stl scale=0.001 0.001 0.001
- link base_link: mass 0.4174748406112292 -> 0.6724614837537145
Joints:
- removed joint Actuator-Knee-Right_Revolute-81
- removed joint Actuator-Left_Revolute-88
- removed joint Actuator-Right_Revolute-87
- removed joint Hip-Left_Rigid-75
- removed joint Hip-Right_Rigid-76
- removed joint Hip-Roll-Actuator-Left_Revolute-68
- removed joint Hip-Roll-control-right_Revolute-67
- removed joint Hip-Spring-Left_Revolute-70
- removed joint Knee-Actuator-Left-1_Revolute-77
- removed joint Random-T_Rigid-61
- removed joint Random-T_Rigid-65
- removed joint Random-T_Rigid-66
- removed joint Shin-Right_Rigid-86
- removed joint Shin-left_Rigid-85
- removed joint Spring-Hip-Right_Revolute-72
- removed joint Spring-Knee-left_Revolute-82
- removed joint Spring-Right_Revolute-78
- removed joint Waist-Pitch-Actuator_Revolute-62
- removed joint Waist-Roll-Actuator_Revolute-64
- removed joint complete_actuator_decoy-v7Mirror_Revolute-71
- removed joint complete_actuator_decoy_Revolute-69
- removed joint holder_hip_2nd-1_Rigid-74
- removed joint holder_hip_2nd-v6Mirror_Rigid-80
- removed joint holder_hip_2ndMirror_Rigid-73
- removed joint holder_hip_2nd_Rigid-79
- removed joint knee_joint_2-v8Mirror_Rigid-83
- removed joint knee_joint_2_Rigid-84
- removed joint waist_Rigid-63
- added joint Ankel_left_Revolute-19: type continuous, parent Ankel_left, child foot_left, origin xyz=-0.038446619999999994 0.0001725500000000002 0.04804246 rpy=-2.1599340154984659e-19 -2.2171418266626333e-19 -2.130031436354674e-19, axis -0.999989 0.004485 0.0011040000000000006
- added joint Ankel_right_Revolute-10: type continuous, parent Ankel_right, child Foot_right, origin xyz=0.0385 0.0 0.048 rpy=-3.141592653589793 -4.690812175909376e-31 8.154403576970184e-32, axis 1.0 0.0 3.4382355471032476e-31
- added joint Hip_Spring_left_Revolute-3: type continuous, parent Hip_Spring_left, child hip_pitch_bracket_right, origin xyz=-0.01649996 3.699999999999981e-05 9.110000000021046e-06 rpy=3.141592653589793 1.5707963267948966 0, axis 0.0005519999999999999 0.002243 -0.999997
- added joint Hip_pitch_left_Revolute-11: type continuous, parent Hip_pitch_left, child Hip_spring_right, origin xyz=0.026879780000000013 0.030117960000000013 0.06735187000000004 rpy=-3.141592653589793 -0.0 -1.1407813263841318e-19, axis 0.999997 0.002243 0.0005520000000000001
- added joint Hip_pitch_right_Revolute-2: type continuous, parent Hip_pitch_right, child Hip_Spring_left, origin xyz=-0.026670080000000002 0.03023804000000001 0.06738140999999999 rpy=5.580160412282723e-19 1.0842021724855044e-19 -1.2763065979448198e-19, axis -0.999997 0.002243 0.000552
- added joint Hip_roll_bracket_right_Rigid-48: type fixed, parent Hip_roll_bracket_right, child knee_right, origin xyz=0.0004410700000000034 0.03865789000000001 0.17581153000000002 rpy=1.9721522630525295e-31 -3.4512664603419266e-31 5.551115123125802e-17
- added joint Hip_spring_right_Revolute-12: type continuous, parent Hip_spring_right, child hip_pitch_bracket_left, origin xyz=0.016499949999999996 3.7000000000000364e-05 9.110000000021046e-06 rpy=-3.141592653589793 -1.5707963267948966 0, axis 0.0005519999999999998 -0.0022429999999999993 0.999997
- added joint Knee_spring_left_Revolute-8: type continuous, parent Knee_spring_left, child knee_brackett_right, origin xyz=-0.014999999999999998 0.0 0.0 rpy=1.4791141972893971e-31 1.5707963267948966 0, axis -2.465190328815662e-31 -5.9164567891575885e-31 -1.0
- added joint Knee_spring_right_Revolute-17: type continuous, parent Knee_spring_right, child knee_brackett_left, origin xyz=0.014999840000000014 6.727000000000206e-05 1.6549999999959653e-05 rpy=-3.141592653589793 -1.5707963267948966 0, axis 0.0011039999999999997 -0.004485 0.999989
- added joint base_link_Rigid-53: type fixed, parent base_link, child Hip_pitch_right, origin xyz=0.05309447999821324 0.026587670011303938 0.6892580900028281 rpy=3.141523771073645 0.0005516016747925701 -0.0022425458152757066
- added joint base_link_Rigid-54: type fixed, parent base_link, child Hip_pitch_left, origin xyz=-0.0866735451213116 0.026559840567045447 0.6892580895544036 rpy=3.141523771073645 0.0005516016747925701 -0.0022425458152757066
- added joint base_link_Rigid-55: type fixed, parent base_link, child IMU-1, origin xyz=-0.025821939089959448 -0.012322293212967468 0.6806080832520717 rpy=-6.888251614786907e-05 0.0005516016747925701 -0.0022425458152757066
- added joint hip_pitch_bracket_left_Rigid-46: type fixed, parent hip_pitch_bracket_left, child hip_roll_acc_left, origin xyz=-0.07286658000000017 -0.017805650000000003 -0.08888396 rpy=-3.141592653589793 1.2037062152420227e-35 -1.3552527156068808e-20
- added joint hip_pitch_bracket_right_Rigid-45: type fixed, parent hip_pitch_bracket_right, child hip_roll_acc_right, origin xyz=-0.07312906000000012 0.018203900000000002 -0.08869976999999998 rpy=-3.141592653589793 6.07576109200659e-39 -1.3552527156068808e-20
- added joint hip_roll_acc_left_Revolute-14: type continuous, parent hip_roll_acc_left, child hip_roll_brackett_left, origin xyz=-0.06300986000000008 0.02640298 -0.020051319999999997 rpy=1.2493735972000932e-19 1.5707963267948966 0, axis -0.004484999999999999 0.9999899999999998 -2.0000000000001113e-06
- added joint hip_roll_acc_right_Revolute-6: type continuous, parent hip_roll_acc_right, child Hip_roll_bracket_right, origin xyz=-0.06254649000000008 -0.026193479999999995 -0.0201 rpy=1.9721522630525295e-31 -1.5707963267948966 0, axis 5.551115123125783e-17 -1.0 1.9721522630525295e-31
- added joint hip_roll_brackett_left_Rigid-49: type fixed, parent hip_roll_brackett_left, child knee_actuator_left, origin xyz=-7.367000000000346e-05 -0.038659050000000014 -0.1758100700000001 rpy=3.1415926535897745 -1.0011929436545832e-18 2.704926097982091e-19
- added joint knee_actuator_left_Revolute-16: type continuous, parent knee_actuator_left, child Knee_spring_right, origin xyz=0.05470685000000112 -0.00025463000000113504 0.06052262000000003 rpy=-3.1415926535897745 -2.0866038768906402e-30 1.112927950723139e-16, axis 0.9999889999999998 0.004484999999999944 0.001104
- added joint knee_brackett_left_Rigid-51: type fixed, parent knee_brackett_left, child Ankel_left, origin xyz=-0.22248103 0.0003116700000000125 -0.06936809000000001 rpy=-5.55107277147842e-17 -1.5707963267948963 0
- added joint knee_brackett_right_Rigid-50: type fixed, parent knee_brackett_right, child Ankel_right, origin xyz=-0.22240434999999997 -1.2490009027033011e-17 0.06958225999999999 rpy=5.551115123125783e-17 -1.5707963267948966 0
- added joint knee_right_Revolute-7: type continuous, parent knee_right, child Knee_spring_left, origin xyz=-0.05464062 -9.409999999999974e-06 0.060582960000000026 rpy=-2.4805977683707598e-31 -6.401791135143172e-31 -1.9311058811127647e-31, axis -1.0 -5.551115123125783e-17 1.9721522630525295e-31
